File: dual-can-gateway.kicad_pcb (KiCad board)
At the start: 2 copper layers, 111.8 x 88.9 mm, 90 parts, among them Q1 AO3401A, Q2 2N7002, U1 STM32F446RETx, U2 STM32F446RETx, U3 ESP32-WROOM-32E, U4 TJA1044GT-3, U5 TJA1044GT-3, U6 TJA1055T, U7 TJA1055T, U8 LM2596S-5, U9 AMS1117-3.3

Commit message: almost done with routing
Parts:
- added ADAM LOGO: ADAM LOGO, Logos:Adam_Logo, F.Cu at (104.1, 90.2)
- added C32: 220 pF, Capacitor_SMD:C_0805_2012Metric, F.Cu at (66.2, 32.3)
- added GND: TestPoint, Connector_PinHeader_2.54mm:PinHeader_1x01_P2.54mm_Vertical, F.Cu at (15.2, 62.7)
- ESP: renamed from U3; value ESP32-WROOM-32E -> ESP32-WROOM-32UE; footprint RF_Module:ESP32-WROOM-32E -> RF_Module:ESP32-WROOM-32UE
- moved STM_1_SWCLK1 106.9 mm to (15.2, 69.1), turned to 180 degrees
- moved STM_1_SWID1 106.7 mm to (15.2, 74.2), turned to 180 degrees
- moved STM_1_NRST1 106.7 mm to (15.2, 71.6), turned to 180 degrees
- moved STM_2_SWCLK1 26.9 mm to (111.8, 69.1)
- moved GND3 22.3 mm to (111.8, 62.2)
- moved STM_2_NRST1 22.3 mm to (111.8, 71.6)
- moved STM_2_SWID1 17.9 mm to (111.8, 74.2)
- moved D2 16.4 mm to (55.3, 32.6), turned to 180 degrees
- moved R7 16.1 mm to (25.2, 17.5), turned to 180 degrees
- moved C31 14.5 mm to (92.3, 80.0), turned to 90 degrees
- moved R1 14.1 mm to (37.6, 87.1)
- moved R8 13.9 mm to (31.0, 72.6), turned to 180 degrees
- moved C1 13.7 mm to (41.5, 80.4)
- moved GND2 13.1 mm to (111.8, 44.3)
- moved ESP_TXD0 13.1 mm to (111.8, 29.8)
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- renumbered U1 to STM_1, U2 to STM_2
Connections:
- net Net-(D1-K) renamed /12V_Raw
- net Net-(D2-K) renamed /5V
- ALWAYS_ON1 pad 1: Net-(Q2-D) -> /<NO NET>
- AUTO_POWER1 pad 1: Net-(Q2-D) -> /<NO NET>
- C1 pad 1: Net-(Q2-D) -> /<NO NET>
- C10 pad 2: Net-(Q2-D) -> /<NO NET>
- C11 pad 2: Net-(Q2-D) -> /<NO NET>
- C12 pad 1: Net-(Q2-D) -> /<NO NET>
- C13 pad 1: Net-(Q2-D) -> /<NO NET>
- C14 pad 1: Net-(D2-A) -> /<NO NET>
- C14 pad 2: Net-(Q1-D) -> /12V_Clean
- C15 pad 1: Net-(U1-VBAT) -> /3.3V
- C15 pad 2: Net-(Q2-D) -> /<NO NET>
- C16 pad 1: Net-(U1-VBAT) -> /3.3V
- C16 pad 2: Net-(Q2-D) -> /<NO NET>
- C17 pad 1: Net-(U1-VBAT) -> /3.3V
- C17 pad 2: Net-(Q2-D) -> /<NO NET>
- C18 pad 1: Net-(U1-VBAT) -> /3.3V
- C18 pad 2: Net-(Q2-D) -> /<NO NET>
- C19 pad 1: Net-(U2-PA3) -> Net-(U2-VDDA)
- C19 pad 2: Net-(Q2-D) -> /<NO NET>
- C2 pad 1: Net-(Q2-D) -> /<NO NET>
- C20 pad 2: Net-(Q2-D) -> /<NO NET>
- C21 pad 1: Net-(Q2-D) -> /3.3V
- C21 pad 2: Net-(Q2-D) -> /<NO NET>
- C22 pad 1: Net-(Q2-D) -> /3.3V
- C22 pad 2: Net-(Q2-D) -> /<NO NET>
- C23 pad 1: Net-(Q2-D) -> /3.3V
- C23 pad 2: Net-(Q2-D) -> /<NO NET>
- C24 pad 1: Net-(Q2-D) -> /3.3V
- C24 pad 2: Net-(Q2-D) -> /<NO NET>
- C25 pad 2: Net-(Q2-D) -> /<NO NET>
- C26 pad 1: Net-(U1-VBAT) -> /3.3V
- C26 pad 2: Net-(Q2-D) -> /<NO NET>
- C27 pad 1: Net-(Q2-D) -> /3.3V
- C27 pad 2: Net-(Q2-D) -> /<NO NET>
- C28 pad 1: Net-(U2-PA3) -> Net-(U2-VDDA)
- C28 pad 2: unconnected-(C28-Pad2) -> /<NO NET>
- C29 pad 2: Net-(Q2-D) -> /<NO NET>
- C3 pad 2: Net-(Q2-D) -> /<NO NET>
- C30 pad 1: Net-(Q2-D) -> /3.3V
- C30 pad 2: Net-(Q2-D) -> /<NO NET>
- C31 pad 1: Net-(Q2-D) -> /3.3V
- C31 pad 2: Net-(Q2-D) -> /<NO NET>
- C4 pad 1: Net-(Q2-D) -> /<NO NET>
- C5 pad 1: Net-(U9-VO) -> /<NO NET>
- C5 pad 2: Net-(U1-VBAT) -> /3.3V
- C6 pad 1: Net-(U1-VBAT) -> /3.3V
- C6 pad 2: Net-(Q2-D) -> /<NO NET>
- C7 pad 2: Net-(Q2-D) -> /<NO NET>
- C8 pad 2: Net-(Q2-D) -> /<NO NET>
- C9 pad 2: Net-(Q2-D) -> /<NO NET>
- D2 pad 2: Net-(D2-A) -> /<NO NET>
- ESP pad 1: Net-(Q2-D) -> /<NO NET>
- ESP pad 15: Net-(Q2-D) -> /<NO NET>
- ESP pad 2: Net-(U1-VBAT) -> /3.3V
- ESP pad 27: Net-(U2-PA2) -> Net-(U2-PA3)
- ESP pad 28: Net-(U2-PA3) -> Net-(U2-PA2)
- ESP pad 30: Net-(U1-PA2) -> Net-(U1-PA3)
- ESP pad 31: Net-(U1-PA3) -> Net-(U1-PA2)
- ESP pad 38: Net-(Q2-D) -> /<NO NET>
- ESP pad 39: Net-(Q2-D) -> /<NO NET>
- FB1 pad 2: Net-(U1-VBAT) -> /3.3V
- FB2 pad 1: Net-(U2-PA3) -> Net-(U2-VDDA)
- FB2 pad 2: Net-(Q2-D) -> /3.3V
- GND1 pad 1: Net-(D2-A) -> /<NO NET>
- GND2 pad 1: Net-(Q2-D) -> /<NO NET>
- GND3 pad 1: Net-(Q2-D) -> /<NO NET>
- ON_OFF1 pad 1: Net-(U8-~{ON}/OFF) -> /<NO NET>
- Q1 pad 3: Net-(Q1-D) -> /12V_Clean
- Q2 pad 2: Net-(Q2-D) -> /<NO NET>
- Q2 pad 3: Net-(Q2-D) -> /<NO NET>
- R10 pad 2: Net-(Q2-D) -> /<NO NET>
- R11 pad 1: Net-(Q2-D) -> /<NO NET>
- R11 pad 2: Net-(Q1-D) -> /12V_Clean
- R12 pad 1: Net-(Q2-D) -> /3.3V
- R12 pad 2: Net-(Q2-D) -> Net-(U2-PB8)
- R7 pad 2: Net-(Q2-D) -> /<NO NET>
- R8 pad 1: Net-(Q2-D) -> Net-(U1-PB12)
- STM_1 pad 1: Net-(U1-VBAT) -> /3.3V
- STM_1 pad 12: Net-(Q2-D) -> /<NO NET>
- STM_1 pad 18: Net-(Q2-D) -> /<NO NET>
- STM_1 pad 19: Net-(U1-VBAT) -> /3.3V
- STM_1 pad 31: Net-(Q2-D) -> /<NO NET>
- STM_1 pad 32: Net-(U1-VBAT) -> /3.3V
- STM_1 pad 33: Net-(Q2-D) -> Net-(U1-PB12)
- STM_1 pad 44: Net-(Q1-D) -> Net-(U1-PA11)
- STM_1 pad 47: Net-(Q2-D) -> /<NO NET>
- STM_1 pad 48: Net-(U1-VBAT) -> /3.3V
- STM_1 pad 63: Net-(Q2-D) -> /<NO NET>
- STM_1 pad 64: Net-(U1-VBAT) -> /3.3V
- STM_2 pad 1: Net-(Q2-D) -> /3.3V
- STM_2 pad 12: Net-(Q2-D) -> /<NO NET>
- STM_2 pad 13: Net-(U2-PA3) -> Net-(U2-VDDA)
- STM_2 pad 18: Net-(Q2-D) -> /<NO NET>
- STM_2 pad 19: Net-(Q2-D) -> /3.3V
- STM_2 pad 31: Net-(Q2-D) -> /<NO NET>
- STM_2 pad 32: Net-(Q2-D) -> /3.3V
- STM_2 pad 47: Net-(Q2-D) -> /<NO NET>
- STM_2 pad 48: Net-(Q2-D) -> /3.3V
- STM_2 pad 61: Net-(Q2-D) -> Net-(U2-PB8)
- STM_2 pad 63: Net-(Q2-D) -> /<NO NET>
- STM_2 pad 64: Net-(Q2-D) -> /3.3V
- U4 pad 2: Net-(Q2-D) -> /<NO NET>
- U4 pad 5: Net-(Q2-D) -> /3.3V
- U4 pad 8: Net-(Q2-D) -> Net-(U2-PB8)
- U5 pad 2: Net-(Q2-D) -> /<NO NET>
- U5 pad 5: Net-(Q2-D) -> /3.3V
- U6 pad 13: Net-(Q2-D) -> /<NO NET>
- U6 pad 14: Net-(Q1-D) -> /12V_Clean
- U6 pad 3: Net-(Q1-D) -> Net-(U1-PA11)
- U6 pad 5: Net-(Q2-D) -> /3.3V
- U6 pad 6: Net-(Q2-D) -> /3.3V
- U7 pad 13: Net-(Q2-D) -> /<NO NET>
- U7 pad 14: Net-(Q1-D) -> /12V_Clean
- U7 pad 5: Net-(Q2-D) -> /3.3V
- U7 pad 6: Net-(Q2-D) -> /3.3V
- U8 pad 1: Net-(Q1-D) -> /12V_Clean
- U8 pad 3: Net-(D2-A) -> /<NO NET>
- U8 pad 5: Net-(U8-~{ON}/OFF) -> /<NO NET>
- U9 pad 1: Net-(D2-A) -> /<NO NET>
- U9 pad 2: Net-(U9-VO) -> /3.3V
Routing:
- net /3.3V: track 0.00 -> 427.0 mm, vias 0 -> 13
- net /5V: track 0.00 -> 172.6 mm, vias 0 -> 6
- net /12V_Clean: track 0.00 -> 107.4 mm, vias 0 -> 5
- net /<NO NET>: track 0.00 -> 105.3 mm, vias 0 -> 51
- net Net-(U2-NRST): track 0.00 -> 87.6 mm, vias 0 -> 2
- net Net-(U1-PA2): track 0.00 -> 77.6 mm
- net Net-(U1-PA3): track 0.00 -> 76.6 mm
- net Net-(U1-PA13): track 0.00 -> 66.1 mm, vias 0 -> 2
- net Net-(U6-INH): track 0.00 -> 63.5 mm, vias 0 -> 4
- net Net-(U2-PB8): track 0.00 -> 54.9 mm, vias 0 -> 2
- net Net-(U1-PA14): track 0.00 -> 51.3 mm, vias 0 -> 2
- net Net-(U2-PA14): track 0.00 -> 49.1 mm, vias 0 -> 2
- net Net-(U2-PA2): track 0.00 -> 41.6 mm
- net Net-(U2-PA3): track 0.00 -> 40.2 mm
- net Net-(U2-PA11): track 0.00 -> 39.7 mm
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- added copper zone on B.Cu, net /<NO NET>
Other:
- board size 111.8 x 88.9 mm -> 101.6 x 88.9 mm
- board text added: "C14"
- board text added: "DCAN_GAT_V10"

Commit message: done with tracing, time to optimize
Parts:
- removed 12V1: 12V, Connector_PinHeader_2.54mm:PinHeader_1x01_P2.54mm_Vertical
- removed ALWAYS_ON1: ALWAYS_ON, Connector_PinHeader_2.54mm:PinHeader_1x01_P2.54mm_Vertical
- removed AUTO_POWER1: AUTO_POWER, Connector_PinHeader_2.54mm:PinHeader_1x01_P2.54mm_Vertical
- removed CAN-FT-H1, CAN-FT-L1, CAN-HS-H1, CAN-HS-L1: LISTEN, Connector_PinHeader_2.54mm:PinHeader_1x01_P2.54mm_Vertical
- removed CAN-FT-H2, CAN-FT-L2, CAN-HS-H2, CAN-HS-L2: MITM, Connector_PinHeader_2.54mm:PinHeader_1x01_P2.54mm_Vertical
- removed GND1: GND, Connector_PinHeader_2.54mm:PinHeader_1x01_P2.54mm_Vertical
- removed ON_OFF1: ON_OFF, Connector_PinHeader_2.54mm:PinHeader_1x01_P2.54mm_Vertical
- added 12V: Conn_01x02_Pin, Connector_PinHeader_2.54mm:PinHeader_1x02_P2.54mm_Vertical, F.Cu at (15.3, 22.9)
- added AUTO_OFF1: Conn_01x02_Pin, Connector_PinHeader_2.54mm:PinHeader_1x02_P2.54mm_Vertical, F.Cu at (15.2, 44.5)
- added CAN-FT-LISTEN1: Conn_01x02_Pin, Connector_PinHeader_2.54mm:PinHeader_1x02_P2.54mm_Vertical, F.Cu at (33.8, 99.1)
- added CAN-FT-MITM1: Conn_01x02_Pin, Connector_PinHeader_2.54mm:PinHeader_1x02_P2.54mm_Vertical, F.Cu at (46.5, 99.1)
- added CAN-HS-LISTEN1: Conn_01x02_Pin, Connector_PinHeader_2.54mm:PinHeader_1x02_P2.54mm_Vertical, F.Cu at (68.6, 99.1)
- added CAN-HS-MITM1: Conn_01x02_Pin, Connector_PinHeader_2.54mm:PinHeader_1x02_P2.54mm_Vertical, F.Cu at (83.8, 99.1)
- U3: renamed from ESP; footprint RF_Module:ESP32-WROOM-32UE -> RF_Module:ESP32-WROOM-32E
- moved R11 11.7 mm to (51.6, 45.7)
- moved C14 5.86 mm to (32.3, 17.5)
- moved U3 3.15 mm to (91.3, 32.7)
- moved R10 0.76 mm to (51.6, 41.1), turned to 180 degrees
- renumbered STM_1 to U1, STM_2 to U2
Connections:
- Q2 pad 3: /<NO NET> -> Net-(AUTO_OFF1-Pin_1)
- R11 pad 1: /<NO NET> -> Net-(AUTO_OFF1-Pin_1)
- U8 pad 5: /<NO NET> -> /AUTO_OFF
Routing:
- net Net-(AUTO_OFF1-Pin_1): track 0.00 -> 59.7 mm
- net /AUTO_OFF: track 0.00 -> 30.0 mm
- net /<NO NET>: track 105.3 -> 78.3 mm, vias 51 -> 49
- net Net-(Q2-G): track 0.00 -> 16.3 mm
- net /3.3V: track 427.0 -> 420.6 mm
- net /5V: track 172.6 -> 167.1 mm
- net Net-(CAN-HS-MITM1-Pin_1): track 29.2 -> 26.9 mm
- net /12V_Clean: track 107.4 -> 105.5 mm, vias 5 -> 4
- net Net-(U2-VCAP_1): track 8.54 -> 9.26 mm
Other:
- board text added: "AUTO_OFF"
- board text added: "CAN-FT-H1"
- board text added: "CAN-FT-H2"
- board text added: "CAN-FT-L1"
- board text added: "CAN-FT-L2"
- board text added: "CAN-HS-H1"
- board text added: "CAN-HS-H2"
- board text added: "CAN-HS-L1"
- board text added: "CAN-HS-L2"
- board text added: "Dual-CAN Filter & Gateway by Hans Lenhard @2026 V1.0"
- board text added: "GND"
- board text removed: "Dual-CAN Filter & Gateway Hans Lenhard @2026 V1.0"

Commit message: proper pins done
Parts:
- removed ESP_EN1, ESP_ID0, ESP_RXD0, ESP_TXD0, JP-MITL-1, JP-MITL-2, JP-MITM-1, JP-MITM-2, STM_1_NRST1, STM_1_SWCLK1, STM_1_SWID1, STM_2_NRST1, STM_2_SWCLK1, STM_2_SWID1: TestPoint, Connector_PinHeader_2.54mm:PinHeader_1x01_P2.54mm_Vertical
- added ESP_FLASH1: Conn_01x04_Pin, Connector_PinHeader_2.54mm:PinHeader_1x04_P2.54mm_Vertical, F.Cu at (111.8, 29.8)
- added JP-HS-LISTEN: Conn_01x02_Pin, Connector_PinHeader_2.54mm:PinHeader_1x02_P2.54mm_Vertical, F.Cu at (63.2, 87.2)
- added JP-HS-MITM: Conn_01x02_Pin, Connector_PinHeader_2.54mm:PinHeader_1x02_P2.54mm_Vertical, F.Cu at (91.2, 87.2)
- added STM_1_FLASH1: Conn_01x03_Pin, Connector_PinHeader_2.54mm:PinHeader_1x03_P2.54mm_Vertical, F.Cu at (15.2, 69.1)
- added STM_2_FLASH1: Conn_01x03_Pin, Connector_PinHeader_2.54mm:PinHeader_1x03_P2.54mm_Vertical, F.Cu at (111.8, 69.1)
Routing:
- net /3.3V: track 420.6 -> 419.2 mm
Other:
- board text added: "ESP_EN1"
- board text added: "ESP_ID0"
- board text added: "ESP_RXD0"
- board text added: "ESP_TXD0"
- board text added: "STM_1_NRST1"
- board text added: "STM_1_SWCLK1"
- board text added: "STM_1_SWID1"
- board text added: "STM_2_NRST1"
- board text added: "STM_2_SWCLK1"
- board text added: "STM_2_SWID1"

Commit message: reworking power input
Connections:
- net /12V_Clean renamed /12V_Switched

Commit message: print ready
Parts:
- removed AUTO_OFF1: Conn_01x02_Pin, Connector_PinHeader_2.54mm:PinHeader_1x02_P2.54mm_Vertical
- added H1: MountingHole_Pad, MountingHole:MountingHole_3.2mm_M3_Pad, F.Cu at (17.3, 17.3)
- added H2: MountingHole_Pad, MountingHole:MountingHole_3.2mm_M3_Pad, F.Cu at (109.7, 17.3)
- added H3: MountingHole_Pad, MountingHole:MountingHole_3.2mm_M3_Pad, F.Cu at (17.3, 97.0)
- added H4: MountingHole_Pad, MountingHole:MountingHole_3.2mm_M3_Pad, F.Cu at (109.7, 97.0)
- added J3: Conn_01x02_Pin, Connector_PinHeader_2.54mm:PinHeader_1x02_P2.54mm_Vertical, F.Cu at (15.2, 41.9)
- added R13: 100k, Resistor_SMD:R_0805_2012Metric, F.Cu at (38.9, 43.9)
- C32: value 220 pF -> 220pF
- D4: value BAT54A -> BAT54C
- moved D4 31.3 mm to (32.4, 41.1), turned to 90 degrees
- moved Q2 25.3 mm to (33.3, 36.0), turned to 90 degrees
- moved R10 24.2 mm to (27.7, 37.1), turned to 0 degrees
- moved R11 23.7 mm to (27.9, 44.5)
- moved D3 18.2 mm to (38.9, 39.3), turned to 180 degrees
- moved D2 9.74 mm to (55.6, 22.9)
- moved C6 7.31 mm to (75.9, 36.1), turned to 0 degrees
- moved U9 5.36 mm to (69.3, 30.7)
- moved ADAM LOGO 4.06 mm to (104.1, 86.1)
- moved C32 3.96 mm to (62.2, 32.3), turned to -90 degrees
- moved L1 3.11 mm to (55.9, 26.9), turned to -90 degrees
- moved C14 2.79 mm to (32.3, 20.3)
- moved STM_1_FLASH1 2.79 mm to (15.2, 66.3)
- moved STM_2_FLASH1 2.79 mm to (111.8, 66.3)
- moved C5 2.07 mm to (75.9, 32.5), turned to 180 degrees
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- renumbered GND2 to GND, GND3 to GND, JP-HS-LISTEN to JP-CAN-HS-LISTEN1, JP-HS-MITM to JP-CAN-HS-MITM1
Connections:
- 12V pad 2: /<NO NET> -> /GND
- C1 pad 1: /<NO NET> -> /GND
- C10 pad 2: /<NO NET> -> /GND
- C11 pad 2: /<NO NET> -> /GND
- C12 pad 1: /<NO NET> -> /GND
- C13 pad 1: /<NO NET> -> /GND
- C14 pad 1: /<NO NET> -> /GND
- C15 pad 2: /<NO NET> -> /GND
- C16 pad 2: /<NO NET> -> /GND
- C17 pad 2: /<NO NET> -> /GND
- C18 pad 2: /<NO NET> -> /GND
- C19 pad 2: /<NO NET> -> /GND
- C2 pad 1: /<NO NET> -> /GND
- C20 pad 2: /<NO NET> -> /GND
- C21 pad 2: /<NO NET> -> /GND
- C22 pad 2: /<NO NET> -> /GND
- C23 pad 2: /<NO NET> -> /GND
- C24 pad 2: /<NO NET> -> /GND
- C25 pad 2: /<NO NET> -> /GND
- C26 pad 2: /<NO NET> -> /GND
- C27 pad 2: /<NO NET> -> /GND
- C28 pad 2: /<NO NET> -> /GND
- C29 pad 2: /<NO NET> -> /GND
- C3 pad 2: /<NO NET> -> /GND
- C30 pad 2: /<NO NET> -> /GND
- C31 pad 2: /<NO NET> -> /GND
- C32 pad 1: /<NO NET> -> /GND
- C4 pad 1: /<NO NET> -> /GND
- C5 pad 1: /<NO NET> -> /GND
- C6 pad 2: /<NO NET> -> /GND
- C7 pad 2: /<NO NET> -> /GND
- C8 pad 2: /<NO NET> -> /GND
- C9 pad 2: /<NO NET> -> /GND
- D2 pad 1: /5V -> Net-(D2-K)
- D2 pad 2: /<NO NET> -> /GND
- D3 pad 1: Net-(U6-INH) -> Net-(U2-PC13)
- D4 pad 1: Net-(Q2-G) -> Net-(U6-INH)
- D4 pad 2: unconnected-(D4-Pad2) -> Net-(D4-Pad2)
- D4 pad 3: Net-(U2-PC13) -> Net-(Q2-G)
- GND pad 1: /<NO NET> -> /GND (x2)
- L1 pad 1: /5V -> Net-(D2-K)
- L1 pad 2: Net-(U9-VI) -> /5V
- Q2 pad 2: /<NO NET> -> /GND
- Q2 pad 3: Net-(AUTO_OFF1-Pin_1) -> Net-(D1-A)
- R10 pad 1: Net-(Q2-G) -> /GND
- R10 pad 2: /<NO NET> -> Net-(Q2-G)
- R11 pad 1: Net-(AUTO_OFF1-Pin_1) -> Net-(D4-Pad2)
- R11 pad 2: /12V_Switched -> Net-(J3-Pin_2)
- R7 pad 1: Net-(D1-A) -> /12V_Raw
- R7 pad 2: /<NO NET> -> Net-(D1-A)
- U1 pad 12: /<NO NET> -> /GND
- U1 pad 18: /<NO NET> -> /GND
- U1 pad 31: /<NO NET> -> /GND
- U1 pad 47: /<NO NET> -> /GND
- U1 pad 63: /<NO NET> -> /GND
- U2 pad 12: /<NO NET> -> /GND
- U2 pad 18: /<NO NET> -> /GND
- U2 pad 31: /<NO NET> -> /GND
- U2 pad 47: /<NO NET> -> /GND
- U2 pad 63: /<NO NET> -> /GND
- U3 pad 1: /<NO NET> -> /GND
- U3 pad 15: /<NO NET> -> /GND
- U3 pad 38: /<NO NET> -> /GND
- U3 pad 39: /<NO NET> -> /GND
- U4 pad 2: /<NO NET> -> /GND
- U5 pad 2: /<NO NET> -> /GND
- U6 pad 13: /<NO NET> -> /GND
- U6 pad 14: /12V_Switched -> /12V_Raw
- U7 pad 13: /<NO NET> -> /GND
- U7 pad 14: /12V_Switched -> /12V_Raw
- U8 pad 2: /5V -> Net-(D2-K)
- U8 pad 3: /<NO NET> -> /GND
- U8 pad 4: unconnected-(U8-FB-Pad4) -> /5V
- U8 pad 5: /AUTO_OFF -> /GND
- U9 pad 1: /<NO NET> -> /GND
- U9 pad 3: Net-(U9-VI) -> /5V
Routing:
- net /12V_Raw: track 13.0 -> 122.1 mm, vias 0 -> 4
- net /12V_Switched: track 105.5 -> 17.7 mm, vias 4 -> 0
- net /<NO NET>: track 78.3 -> 0.00 mm, vias 49 -> 0
- net /GND: track 0.00 -> 78.2 mm, vias 0 -> 47
- net Net-(AUTO_OFF1-Pin_1): track 59.7 -> 0.00 mm
- net Net-(D2-K): track 0.00 -> 36.9 mm
- net /AUTO_OFF: track 30.0 -> 0.00 mm
- net Net-(U6-INH): track 63.3 -> 45.8 mm
- net Net-(D1-A): track 10.9 -> 23.4 mm, vias 0 -> 2
- net Net-(U2-PC13): track 27.6 -> 39.5 mm
- net Net-(J3-Pin_2): track 0.00 -> 11.8 mm
- net Net-(U1-PC13): track 36.0 -> 26.0 mm
- net Net-(U9-VI): track 9.48 -> 0.00 mm
- net Net-(D4-Pad2): track 0.00 -> 6.29 mm
- net /3.3V: track 419.2 -> 422.8 mm
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- added copper zone on B.Cu, net /GND
- removed copper zone on B.Cu, net /<NO NET>
Other:
- board text added: "ALWAYS_ON"
- board text added: "Dual-CAN Filter & Gateway by Hans Lenhard - 2026 - V1.0"
- board text removed: "AUTO_OFF"
- board text removed: "Dual-CAN Filter & Gateway by Hans Lenhard @2026 V1.0"

Commit message: updated logo
Parts:
- removed ADAM LOGO: ADAM LOGO, Logos:Adam_Logo
- added G***: LOGO, Logos:logo_lhe, F.Cu at (105.2, 84.6)
- moved D2 7.08 mm to (62.5, 24.6), turned to 90 degrees
Routing:
- net Net-(D2-K): track 36.9 -> 38.4 mm
Other:
- board text added: "Dual-CAN Gateway"
- board text added: "Hans Lenhard 2026 - V1.0"
- board text added: "LHE_DCANGW_10"
- board text removed: "DCAN_GAT_V10"
- board text removed: "Dual-CAN Filter & Gateway by Hans Lenhard - 2026 - V1.0"

Commit message: v1.1
Parts:
- D1: value D_Zener -> MMSZ12T1G
- L1: footprint Inductor_THT:L_Radial_D8.7mm_P5.00mm_Fastron_07HCP -> Inductor_SMD:L_Bourns_SRP6060FA
- R9: value R -> 10k
- moved D2 10.8 mm to (51.7, 23.5), turned to 0 degrees
- moved L1 4.36 mm to (55.1, 31.2)
Routing:
- net Net-(D2-K): track 38.4 -> 32.8 mm
- net /5V: track 165.6 -> 161.8 mm
- net /12V_Raw: track 122.1 -> 120.8 mm
Other:
- board text added: "ESP_EN"
- board text added: "ESP_ID"
- board text added: "ESP_RXD"
- board text added: "ESP_TXD"
- board text added: "Hans Lenhard 2026 - V1.1"
- board text added: "LHE_DCANGW_11"
- board text added: "STM_1_NRST"
- board text added: "STM_1_SWCLK"
- board text added: "STM_1_SWID"
- board text added: "STM_2_NRST"
- board text added: "STM_2_SWCLK"
- board text added: "STM_2_SWID"
- board text removed: "ESP_EN1"
- board text removed: "ESP_ID0"
- board text removed: "ESP_RXD0"
- board text removed: "ESP_TXD0"
- board text removed: "Hans Lenhard 2026 - V1.0"
- board text removed: "LHE_DCANGW_10"
- board text removed: "STM_1_NRST1"
- board text removed: "STM_1_SWCLK1"
- board text removed: "STM_1_SWID1"
- board text removed: "STM_2_NRST1"
- board text removed: "STM_2_SWCLK1"
- board text removed: "STM_2_SWID1"

Commit message: small adjustment
Parts:
- moved R5 0.28 mm to (63.3, 95.4)
Changed lines of the file:
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@@
 	(footprint "Resistor_SMD:R_0805_2012Metric"
 		(layer "F.Cu")
-		(at 91.212 95.4005 90)
+		(at 91.212 95.377 90)
 		(descr "Resistor SMD 0805 (2012 Metric), square (rectangular) end terminal, IPC-7351 nominal, (Body size source: IPC-SM-782 page 72, https://www.pcb-3d.com/wordpress/wp-content/uploads/ipc-sm-782a_amendment_1_and_2.pdf)")
 		(tags "resistor")
@@
 	(footprint "Resistor_SMD:R_0805_2012Metric"
 		(layer "F.Cu")
-		(at 63.272 95.6545 -90)
+		(at 63.272 95.377 -90)
 		(descr "Resistor SMD 0805 (2012 Metric), square (rectangular) end terminal, IPC-7351 nominal, (Body size source: IPC-SM-782 page 72, https://www.pcb-3d.com/wordpress/wp-content/uploads/ipc-sm-782a_amendment_1_and_2.pdf)")
 		(tags "resistor")
@@
 	)
 	(segment
-		(start 68.58 99.06)
-		(end 65.765 99.06)
+		(start 66.0425 99.06)
+		(end 63.5495 96.567)
 		(width 0.3)
 		(layer "F.Cu")
@@
 	)
 	(segment
-		(start 70.4088 82.8548)
-		(end 70.7136 82.55)
+		(start 68.58 99.06)
+		(end 66.0425 99.06)
 		(width 0.3)
 		(layer "F.Cu")
@@
 	)
 	(segment
-		(start 68.58 88.4428)
-		(end 70.4088 86.614)
+		(start 70.7136 82.55)
+		(end 70.4088 82.8548)
 		(width 0.3)
 		(layer "F.Cu")
@@
 	)
 	(segment
-		(start 68.58 99.06)
-		(end 68.58 88.4428)
+		(start 70.4088 82.8548)
+		(end 70.4088 86.614)
 		(width 0.3)
 		(layer "F.Cu")
@@
 	)
 	(segment
-		(start 70.4088 86.614)
-		(end 70.4088 82.8548)
+		(start 72.39 82.55)
+		(end 70.7136 82.55)
 		(width 0.3)
 		(layer "F.Cu")
@@
 	)
 	(segment
-		(start 65.765 99.06)
-		(end 63.272 96.567)
+		(start 68.58 88.4428)
+		(end 68.58 99.06)
 		(width 0.3)
 		(layer "F.Cu")
@@
 	)
 	(segment
-		(start 70.7136 82.55)
-		(end 72.39 82.55)
+		(start 70.4088 86.614)
+		(end 68.58 88.4428)
 		(width 0.3)
 		(layer "F.Cu")
