File: dual-can-gateway.kicad_sch (KiCad schematic)
At the start: 90 parts, among them Q1 AO3401A, Q2 2N7002, U1 STM32F446RETx, U2 STM32F446RETx, U3 ESP32-WROOM-32E, U4 TJA1044GT-3, U5 TJA1044GT-3, U6 TJA1055T, U7 TJA1055T, U8 LM2596S-5, U9 AMS1117-3.3

Commit message: almost done with routing
Parts:
- added C32: 220 pF, Capacitor_SMD:C_0805_2012Metric, symbol Device:C
- U3: value ESP32-WROOM-32E -> ESP32-WROOM-32UE
Connections:
- net 3.3V: now reaches C15.1, C16.1, C17.1, C18.1, C26.1, C5.2, C6.1, FB1.2, U1.1 (VBAT), U1.19 (VDD), U1.32 (VDD), U1.48 (VDD), U1.64 (VDD), U3.2 (VDD)
- net 3.3V: now also C21.1, C22.1, C23.1, C24.1, C27.1, C30.1, C31.1, FB2.2, R12.1, U2.1 (VBAT), U2.19 (VDD), U2.32 (VDD), U2.48 (VDD), U2.64 (VDD), U4.5 (VIO), U5.5 (VIO), U6.5 (~{STB}), U6.6 (EN), U7.5 (~{STB}), U7.6 (EN), U9.2 (VO)
- net at ALWAYS_ON1.1, AUTO_POWER1.1, C1.1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: no longer names the net of ALWAYS_ON1.1, AUTO_POWER1.1, C1.1, C10.2, C11.2, C12.1, C13.1, C15.2, C16.2, C17.2, C18.2, C19.2, C2.1, C20.2, C21.2, C22.2, C23.2, C24.2, C25.2, C26.2, C27.2, C29.2, C3.2, C30.2, C31.2, C4.1, C6.2, C7.2, C8.2, C9.2, GND2.1, GND3.1, Q2.2 (S), Q2.3 (D), R10.2, R11.1, R7.2, U1.12 (VSSA), U1.18 (VSS), U1.31 (VSS), U1.47 (VSS), U1.63 (VSS), U2.12 (VSSA), U2.18 (VSS), U2.31 (VSS), U2.47 (VSS), U2.63 (VSS), U3.[1,15,38,39] (GND), U4.2 (GND), U5.2 (GND), U6.13 (GND), U7.13 (GND)
- net at ALWAYS_ON1.1, AUTO_POWER1.1, C1.1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: now also C14.1, C28.2, C5.1, D2.2 (A), GND1.1, ON_OFF1.1, U8.3 (GND), U8.5 (~{ON}/OFF), U9.1 (GND), C32.1; no longer C21.1, C22.1, C23.1, C24.1, C27.1, C30.1, C31.1, FB2.2, R12.1, R12.2, R8.1, U1.33 (PB12), U2.1 (VBAT), U2.19 (VDD), U2.32 (VDD), U2.48 (VDD), U2.61 (PB8), U2.64 (VDD), U4.5 (VIO), U4.8 (S), U5.5 (VIO), U6.5 (~{STB}), U6.6 (EN), U7.5 (~{STB}), U7.6 (EN)
- net 5V: now reaches C1.2, C2.2, C3.1, C4.2, D2.1 (K), L1.1, U4.3 (VCC), U5.3 (VCC), U6.10 (VCC), U7.10 (VCC), U8.2 (OUT)
- net 5V: now also C32.2
- net at C19.1, C28.1, FB2.1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: no longer U2.17 (PA3), U3.28 (IO17)
- net at U2.16 (PA2): now also U3.28 (IO17); no longer U3.27 (IO16)
- net 12V_Raw: now reaches 12V1.1, D1.1 (K), Q1.2 (S)
- net 12V_Clean: now reaches C14.2, Q1.3 (D), R11.2, U6.14 (BAT), U7.14 (BAT), U8.1 (VIN)
- net 12V_Clean: no longer U1.44 (PA11), U6.3 (RXD)
- net at U3.30 (IO18): now also U1.17 (PA3); no longer U1.16 (PA2)
- net at U3.31 (IO19): now also U1.16 (PA2); no longer U1.17 (PA3)
- new net: R12.2, U2.61 (PB8), U4.8 (S)
- new net: U2.17 (PA3), U3.27 (IO16)
- new net: U1.44 (PA11), U6.3 (RXD)
- new net: R8.1, U1.33 (PB12)
Other:
- note removed: "GND"
- moved on the sheet: C19, C28, C5

Commit message: done with tracing, time to optimize
Parts:
- removed 12V1: 12V, Connector_PinHeader_2.54mm:PinHeader_1x01_P2.54mm_Vertical, symbol Connector:TestPoint
- removed ALWAYS_ON1: ALWAYS_ON, Connector_PinHeader_2.54mm:PinHeader_1x01_P2.54mm_Vertical, symbol Connector:TestPoint
- removed AUTO_POWER1: AUTO_POWER, Connector_PinHeader_2.54mm:PinHeader_1x01_P2.54mm_Vertical, symbol Connector:TestPoint
- removed CAN-FT-H1, CAN-FT-L1, CAN-HS-H1, CAN-HS-L1: LISTEN, Connector_PinHeader_2.54mm:PinHeader_1x01_P2.54mm_Vertical, symbol Connector:TestPoint
- removed CAN-FT-H2, CAN-FT-L2, CAN-HS-H2, CAN-HS-L2: MITM, Connector_PinHeader_2.54mm:PinHeader_1x01_P2.54mm_Vertical, symbol Connector:TestPoint
- removed GND1: GND, Connector_PinHeader_2.54mm:PinHeader_1x01_P2.54mm_Vertical, symbol Connector:TestPoint
- removed ON_OFF1: ON_OFF, Connector_PinHeader_2.54mm:PinHeader_1x01_P2.54mm_Vertical, symbol Connector:TestPoint
- added AUTO_OFF1, CAN-FT-LISTEN1, CAN-FT-MITM1, CAN-HS-LISTEN1, CAN-HS-MITM1, J1: Conn_01x02_Pin, Connector_PinHeader_2.54mm:PinHeader_1x02_P2.54mm_Vertical, symbol Connector:Conn_01x02_Pin
Connections:
- net 12V_Raw: now also J1.1 (Pin_1)
- net at R5.2, U4.6 (CANL): now also CAN-HS-LISTEN1.1 (Pin_1)
- net at C1.1, C10.2, C11.2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: now also J1.2 (Pin_2); no longer Q2.3 (D), R11.1, U8.5 (~{ON}/OFF)
- net at JP-MITL-1.1, U4.7 (CANH): now also CAN-HS-LISTEN1.2 (Pin_2)
- net at C8.1, R2.1, U6.12 (CANL): now also CAN-FT-LISTEN1.1 (Pin_1)
- net at C9.1, R1.1, U6.11 (CANH): now also CAN-FT-LISTEN1.2 (Pin_2)
- net at R6.1, U5.6 (CANL): now also CAN-HS-MITM1.1 (Pin_1)
- net at JP-MITM-1.1, U5.7 (CANH): now also CAN-HS-MITM1.2 (Pin_2)
- net at C11.1, R3.1, U7.11 (CANH): now also CAN-FT-MITM1.2 (Pin_2)
- net at C10.1, R4.1, U7.12 (CANL): now also CAN-FT-MITM1.1 (Pin_1)
- new net: AUTO_OFF1.1 (Pin_1), Q2.3 (D), R11.1
- new net AUTO_OFF: AUTO_OFF1.2 (Pin_2), U8.5 (~{ON}/OFF)
Other:
- moved on the sheet: C11, D4

Commit message: proper pins done
Parts:
- removed ESP_EN1, ESP_ID0, ESP_RXD0, ESP_TXD0, JP-MITL-1, JP-MITL-2, JP-MITM-1, JP-MITM-2, STM_1_NRST1, STM_1_SWCLK1, STM_1_SWID1, STM_2_NRST1, STM_2_SWCLK1, STM_2_SWID1: TestPoint, Connector_PinHeader_2.54mm:PinHeader_1x01_P2.54mm_Vertical, symbol Connector:TestPoint
- added ESP_FLASH1: Conn_01x04_Pin, Connector_PinHeader_2.54mm:PinHeader_1x04_P2.54mm_Vertical, symbol Connector:Conn_01x04_Pin
- added JP-CAN-HS-LISTEN1, JP-CAN-HS-MITM1: Conn_01x02_Pin, Connector_PinHeader_2.54mm:PinHeader_1x02_P2.54mm_Vertical, symbol Connector:Conn_01x02_Pin
- added STM_1_FLASH1, STM_2_FLASH1: Conn_01x03_Pin, Connector_PinHeader_2.54mm:PinHeader_1x03_P2.54mm_Vertical, symbol Connector:Conn_01x03_Pin
Connections:
- net at R5.1: now also JP-CAN-HS-LISTEN1.2 (Pin_2)
- net at U1.49 (PA14): now also STM_1_FLASH1.1 (Pin_1)
- net at CAN-HS-LISTEN1.2 (Pin_2), U4.7 (CANH): now also JP-CAN-HS-LISTEN1.1 (Pin_1)
- net at U2.46 (PA13): now also STM_2_FLASH1.3 (Pin_3)
- net at U3.34 (RXD0/IO3): now also ESP_FLASH1.2 (Pin_2)
- net at U2.7 (NRST): now also STM_2_FLASH1.2 (Pin_2)
- net at U2.49 (PA14): now also STM_2_FLASH1.1 (Pin_1)
- net at U3.35 (TXD0/IO1): now also ESP_FLASH1.1 (Pin_1)
- net at U1.46 (PA13): now also STM_1_FLASH1.3 (Pin_3)
- net at U3.3 (EN): now also ESP_FLASH1.3 (Pin_3)
- net at R6.2: now also JP-CAN-HS-MITM1.2 (Pin_2)
- net at U3.25 (IO0): now also ESP_FLASH1.4 (Pin_4)
- net at CAN-HS-MITM1.2 (Pin_2), U5.7 (CANH): now also JP-CAN-HS-MITM1.1 (Pin_1)
- net at U1.7 (NRST): now also STM_1_FLASH1.2 (Pin_2)

Commit message: reworking power input
Parts:
- removed AUTO_OFF1: Conn_01x02_Pin, Connector_PinHeader_2.54mm:PinHeader_1x02_P2.54mm_Vertical, symbol Connector:Conn_01x02_Pin
- added J2: Conn_01x03_Pin, symbol Connector:Conn_01x03_Pin
Connections:
- net 12V_Raw: now also R7.1
- net 5V: now also L1.2, U9.3 (VI); no longer D2.1 (K), L1.1, U8.2 (OUT)
- net AUTO_OFF: no longer U8.5 (~{ON}/OFF)
- net at C1.1, C10.2, C11.2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: now also Q2.1 (G), U8.5 (~{ON}/OFF); no longer Q2.2 (S), R7.2
- net at D3.1: no longer U6.1 (INH)
- net at D3.2: no longer U1.2 (PC13)
- net at D1.2 (A), Q1.1 (G): now also Q2.3 (D), R7.2; no longer R7.1
- net at U2.2 (PC13): no longer D4.3
- net at R11.1: now also J2.1 (Pin_1); no longer Q2.3 (D)
- net 12V_Clean renamed 12V_Switched
- new net: D2.1 (K), L1.1, U8.2 (OUT)
- new net: Q2.2 (S), R10.1
- now unconnected: D3.3, D4.1
Other:
- note added: "12V_Switched"
- note removed: "12V Clean"
- moved on the sheet: C32, D1, D3, D4, Q1, Q2, R10, R7, U9

Commit message: print ready
Parts:
- removed D4: BAT54A, Package_TO_SOT_SMD:SOT-23, symbol Diode:BAT54A
- removed J2: Conn_01x03_Pin, symbol Connector:Conn_01x03_Pin
- added D4: BAT54C, Package_TO_SOT_SMD:SOT-23, symbol Diode:BAT54C
- added H1, H2, H3, H4: MountingHole_Pad, MountingHole:MountingHole_3.2mm_M3_Pad, symbol Mechanical:MountingHole_Pad
- added J3: Conn_01x02_Pin, Connector_PinHeader_2.54mm:PinHeader_1x02_P2.54mm_Vertical, symbol Connector:Conn_01x02_Pin
- added R13: 100k, Resistor_SMD:R_0805_2012Metric, symbol Device:R
- C32: value 220 pF -> 220pF
Connections:
- net 12V_Raw: now also U6.14 (BAT), U7.14 (BAT), J3.1 (Pin_1)
- net 12V_Switched: no longer R11.2, U6.14 (BAT), U7.14 (BAT)
- net 5V: now also U8.4 (FB)
- net GND: now reaches C1.1, C10.2, C11.2, C12.1, C13.1, C14.1, C15.2, C16.2, C17.2, C18.2, C19.2, C2.1, C20.2, C21.2, C22.2, C23.2, C24.2, C25.2, C26.2, C27.2, C28.2, C29.2, C3.2, C30.2, C31.2, C32.1, C4.1, C5.1, C6.2, C7.2, C8.2, C9.2, D2.2 (A), GND2.1, GND3.1, J1.2 (Pin_2), U1.12 (VSSA), U1.18 (VSS), U1.31 (VSS), U1.47 (VSS), U1.63 (VSS), U2.12 (VSSA), U2.18 (VSS), U2.31 (VSS), U2.47 (VSS), U2.63 (VSS), U3.[1,15,38,39] (GND), U4.2 (GND), U5.2 (GND), U6.13 (GND), U7.13 (GND), U8.3 (GND), U8.5 (~{ON}/OFF), U9.1 (GND)
- net GND: now also Q2.2 (S), R10.1, R13.2; no longer Q2.1 (G), R10.2
- net at D3.1: now also U2.2 (PC13)
- net at D3.2: now also U1.2 (PC13)
- net at D3.3: now also Q2.1 (G), R10.2, D4.3
- net at R11.1: now also D4.2
- net at U6.1 (INH): now also D4.1, R13.1
- new net: J3.2 (Pin_2), R11.2
Other:
- note added: "JP_ALWAYS_ON"
- note removed: "12V_Switched"
- moved on the sheet: C32, D3, Q1

Commit message: updated readme
Other:
- company: ADAM Hardware Engine -> dexus1337
Changed lines of the file:
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@@
 	(title_block
 		(title "Automotive Dual-CAN Filter & WiFi Gateway")
-		(company "ADAM Hardware Engine")
+		(company "dexus1337")
 		(comment 1 "2x STM32F446 + ESP32 + 2x TJA1055 + 2x TJA1051")
 	)

Commit message: v1.1
Parts:
- D1: value D_Zener -> MMSZ12T1G
- L1: footprint Inductor_THT:L_Radial_D8.7mm_P5.00mm_Fastron_07HCP -> Inductor_SMD:L_Bourns_SRP6060FA
- R9: value R -> 10k
- renumbered J1 to 12V1
Changed lines of the file:
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@@
 			)
 		)
-		(property "Value" "R"
+		(property "Value" "10k"
 			(at 109.22 227.33 90)
 			(show_name no)
@@
 			)
 		)
-		(property "Footprint" "Inductor_THT:L_Radial_D8.7mm_P5.00mm_Fastron_07HCP"
+		(property "Footprint" "Inductor_SMD:L_Bourns_SRP6060FA"
 			(at 95.25 39.37 0)
 			(hide yes)
@@
 			)
 		)
-		(property "Value" "D_Zener"
+		(property "Value" "MMSZ12T1G"
 			(at 36.83 24.892 0)
 			(show_name no)
@@
 		(dnp no)
 		(fields_autoplaced yes)
-		(property "Reference" "J1"
+		(property "Reference" "12V1"
 			(at 18.415 35.56 0)
 			(hide yes)
@@
 			(project "dual-can-gateway"
 				(path "/00000000-0000-0000-0000-000064d1a2f1"
-					(reference "J1")
+					(reference "12V1")
 					(unit 1)
 				)

Commit message: hopefully fixed auto wake/shutdown
Parts:
- added R14, R15: 10k, Resistor_SMD:R_0805_2012Metric, symbol Device:R
- R11: value 100k -> 10k
Connections:
- net 3.3V: no longer U6.5 (~{STB}), U6.6 (EN)
- net GND: now also R14.1, R15.2
- net at U1.38 (PC7): now also U6.5 (~{STB}), R15.1
- net at U1.39 (PC8): now also U6.6 (EN), R14.2
