File: automotive-gateway.kicad_pcb (KiCad board)
At the start: 2 copper layers, 101.6 x 88.9 mm, 103 parts, among them J3 Conn_01x02_Pin, Q1 AO3401A, Q2 2N7002, U1 STM32F405RGTx, U10 TJA1021xT, U11 TJA1021xT, U2 STM32F405RGTx, U3 ESP32-WROOM-32UE, U4 TJA1044GT-3, U5 TJA1044GT-3, U6 TJA1055T/3, U7 TJA1055T/3, U8 LM2596S-5, U9 AMS1117-3.3

Commit message: Add AG (Automotive Gateway) logo footprints and update PCB silkscreen
- Created logo_ag.kicad_mod (10mm) and size variants: 6mm, 8mm, 12mm, 14mm
- Created clean vector SVG exports (LOGO_AG.svg, LOGO_AG_12mm.svg)
- Preserved exact motorsport/OEM styling, 45-degree forward slant, and ribbon stroke weights
- Updated silkscreen logo on automotive-gateway.kicad_pcb to logo_ag_12mm
Parts:
- G***: value LOGO_DUAL_CAN -> LOGO_AG; footprint mylib:logo_dual_can_12mm -> mylib:logo_ag_12mm
Changed lines of the file:
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@@
 		)
 	)
-	(footprint "mylib:logo_dual_can_12mm"
+	(footprint "mylib:logo_ag_12mm"
 		(layer "F.Cu")
 		(at 71.0692 20.2946)
@@
 			)
 		)
-		(property "Value" "LOGO_DUAL_CAN"
+		(property "Value" "LOGO_AG"
 			(at 0 0 0)
 			(layer "F.SilkS")
@@
 		(fp_poly
 			(pts
-				(xy -2.2759 -3.8069) (xy 0.1793 -3.8069) (xy -0.5655 -2.7034) (xy -2.9931 -2.7034) (xy -2.2759 -3.8069)
+				(xy -2.2396 -3.8157) (xy -1.0783 -3.8157) (xy -0.4424 -2.6544) (xy -1.0783 -1.6866) (xy -1.6590 -2.6820) (xy -2.4055 -2.6820) (xy -5.4194 2.6820) (xy -6.0000 1.6590) (xy -2.2396 -3.8157)
 			)
 			(stroke
@@
 		(fp_poly
 			(pts
-				(xy 0.3724 2.5931) (xy 2.9931 2.5931) (xy 2.2207 3.7793) (xy -0.4 3.7793) (xy 0.3724 2.5931)
+				(xy 1.0783 -3.8157) (xy 5.9724 -3.8157) (xy 5.2811 -2.7097) (xy 1.2719 -2.7097) (xy -0.6359 0.1659) (xy -1.9355 0.1659) (xy 0.3594 -3.3733) (xy 0.7189 -3.6774) (xy 1.0783 -3.8157)
 			)
 			(stroke
@@
 		(fp_poly
 			(pts
-				(xy 1.0897 -3.8069) (xy 5.9724 -3.8069) (xy 5.2276 -2.7034) (xy 1.2552 -2.7034) (xy -1.3931 1.3241)
-				(xy -1.669 1.5724) (xy -1.9448 1.6552) (xy -6 1.6552) (xy -3.6828 -1.7103) (xy -2.3586 -1.7103)
-				(xy -3.8759 0.5241) (xy -2.2483 0.5517) (xy 0.3172 -3.3379) (xy 0.6483 -3.6414) (xy 1.0897 -3.8069)
+				(xy -2.0184 -2.2396) (xy -1.9078 -2.2396) (xy -1.3825 -1.2166) (xy -1.8525 -0.4977) (xy -2.0184 -0.7189) (xy -2.7097 0.5530) (xy -0.4424 0.5530) (xy 1.3272 3.7880) (xy 0.1659 3.7880) (xy -0.9401 1.6590) (xy -3.2627 1.6590) (xy -4.3687 3.7880) (xy -5.5023 3.7880) (xy -3.7880 0.6636) (xy -2.0184 -2.2396)
 			)
 			(stroke
@@
 		(fp_poly
 			(pts
-				(xy 2.0828 -1.9586) (xy 5.9724 -1.9586) (xy 3.7379 1.4069) (xy 2.4138 1.3793) (xy 3.9034 -0.8) (xy 2.1655 -0.8276)
-				(xy -0.4828 3.2276) (xy -0.869 3.6138) (xy -1.2552 3.7793) (xy -5.9724 3.7793) (xy -5.2 2.5931)
-				(xy -1.4207 2.5931) (xy 1.3931 -1.6828) (xy 1.6414 -1.8759) (xy 2.0828 -1.9586)
+				(xy 2.5438 -1.9355) (xy 4.7834 -1.9355) (xy 4.0645 -0.8295) (xy 2.1843 -0.8295) (xy 1.4654 0.2488) (xy 0.8571 -0.8571) (xy 1.5760 -1.8249) (xy 1.8249 -1.9355) (xy 2.5438 -1.9355)
 			)
 			(stroke
+				(width 0)
+				(type solid)
+			)
+			(fill yes)
+			(layer "F.SilkS")
+		)
+		(fp_poly
+			(pts
+				(xy 0.4699 -0.9954) (xy 2.5161 2.6820) (xy 2.9862 2.6820) (xy 4.0369 1.0230) (xy 1.8525 1.0230) (xy 2.5438 -0.0829) (xy 5.8341 -0.0829) (xy 5.9724 0.0000) (xy 3.6774 3.5392) (xy 3.2350 3.7880) (xy 2.1567 3.7880) (xy 1.6313 3.3456) (xy -0.1935 0.0276) (xy 0.4699 -0.9954)
+			)
+			(stroke
