File: automotive-gateway.kicad_sch (KiCad schematic)
At the start: 101 parts, among them J3 Conn_01x02_Pin, Q1 AO3401A, Q2 2N7002, U1 STM32F405RGTx, U10 TJA1021xT, U11 TJA1021xT, U2 STM32F405RGTx, U3 ESP32-WROOM-32UE, U4 TJA1044GT-3, U5 TJA1044GT-3, U6 TJA1055T/3, U7 TJA1055T/3, U8 LM2596S-5, U9 AMS1117-3.3

Commit message: added external clock source
Parts:
- added C40, C41, C42, C43: 15pF, Capacitor_SMD:C_0805_2012Metric, symbol Device:C
- added Y1, Y2: Crystal_GND24_Small, Crystal:Crystal_SMD_3225-4Pin_3.2x2.5mm_HandSoldering, symbol Device:Crystal_GND24_Small
Connections:
- net GND: now also C40.1, C41.1, C42.1, C43.1, Y1.2 (G), Y1.4 (G), Y2.2 (G), Y2.4 (G)
- net at U1.5 (PH0): now also C41.2, Y1.1
- net at U1.6 (PH1): now also C40.2, Y1.3
- net at U2.5 (PH0): now also C42.2, Y2.1
- net at U2.6 (PH1): now also C43.2, Y2.3
